File: Night_Light.kicad_pcb (KiCad board)
At the start: 2 copper layers, 25.4 x 25.4 mm, 6 parts, among them J1 3V0, Q1 2N3904

Commit message: Add mark and name
Other:
- board text added: "Dribin"
- board text added: "Zach"
- board text added: "{dblquote}Chef{dblquote}"
Changed lines of the file:
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@@
     )
   )
+  (gr_rect (start 130.81 79.502) (end 129.286 77.978) (layer "B.SilkS") (width 0.15) (fill none))
+  (gr_rect (start 130.429 78.359) (end 129.667 79.121) (layer "B.SilkS") (width 0.15) (fill none))
+  (gr_poly
+    (pts
+      (xy 130.81 78.74)
+      (xy 130.048 79.502)
+      (xy 129.286 78.74)
+      (xy 130.048 77.978)
+    ) (layer "B.SilkS") (width 0.15) (fill none))
+  (gr_circle (center 130.048 78.74) (end 130.556 77.724) (layer "B.SilkS") (width 0.15) (fill none))
   (gr_line (start 124.46 88.9) (end 157.607 88.9) (layer "Cmts.User") (width 0.15))
   (gr_line (start 139.7 73.66) (end 139.7 106.68) (layer "Cmts.User") (width 0.15))
@@
   )
   (gr_text "Designed by a\nJulian Jayhawk" (at 139.7 84.074) (layer "B.SilkS")
+    (effects (font (size 1 1) (thickness 0.15)) (justify mirror))
+  )
+  (gr_text "Zach" (at 130.048 81.28) (layer "B.SilkS")
+    (effects (font (size 1 1) (thickness 0.15)) (justify mirror))
+  )
+  (gr_text "{dblquote}Chef{dblquote}" (at 130.048 82.804) (layer "B.SilkS")
+    (effects (font (size 1 1) (thickness 0.15)) (justify mirror))
+  )
+  (gr_text "Dribin" (at 130.048 84.328) (layer "B.SilkS")
     (effects (font (size 1 1) (thickness 0.15)) (justify mirror))
   )
@@
     )
   )
+  (group "" (id 29f702bd-cddf-4c33-ad47-a58123ba37fc)
+    (members
+      3f045c61-038a-4641-85f2-d00c5a3f9458
+      88b0fa61-f556-4cdc-ad67-906578bdb9ce
+      da8a18e7-03aa-4329-8b27-90dd7242f5f6
+      fc1fbaae-408a-42b0-8805-42142fc55472
+    )
+  )
